File: Circuit/mic_preamp_v1.kicad_pcb (KiCad board)
At the start: 2 copper layers, 67.3 x 58.4 mm, 22 parts, among them J1 AudioJack2, J2 Barrel_Jack_Switch, J3 Conn_Coaxial, U1 LM358, U2 L7805

Commit message: Finish circuit
Parts:
- C1, C2, C3, C4, C5, C6, C7, D1, D2, R1, R2, R3, R4, R5, R6, R7, R8, U2: moved to B.Cu
- moved J1 18.5 mm to (166.9, 96.5)
- moved J3 7.10 mm to (136.6, 96.5)
- moved U2 5.24 mm to (166.6, 83.6), turned to 90 degrees
- moved R2 0.72 mm to (152.0, 108.5)
Routing:
- net Net-(D1-K): track 39.4 -> 48.6 mm
- net +5V: track 91.9 -> 93.4 mm
- net Net-(C1-Pad2): track 20.8 -> 21.9 mm
- net Net-(C4-Pad2): track 11.0 -> 10.1 mm
Other:
- board size 67.3 x 58.4 mm -> 67.3 x 61 mm
